Commit message: Add on/off sensors via yaml, updated turtlebot3.urdf.xacro

File: robot_description/urdf/realsence_d435.xacro (robot description, xacro)
@@ -1,159 +1,15 @@
 <?xml version="1.0"?>
-<!--
-# Copyright 2023 Intel Corporation. All Rights Reserved.
-#
-# Licensed under the Apache License, Version 2.0 (the "License");
-# you may not use this file except in compliance with the License.
-# You may obtain a copy of the License at
-#
-#     http://www.apache.org/licenses/LICENSE-2.0
-#
-# Unless required by applicable law or agreed to in writing, software
-# distributed under the License is distributed on an "AS IS" BASIS,
-# WITHOUT WARRANTIES OR CONDITIONS OF ANY KIND, either express or implied.
-# See the License for the specific language governing permissions and
-# limitations under the License.
--->
-<!--
-This is the URDF model for the Intel RealSense 430 camera, in its
-aluminum peripherial evaluation case.
--->
-<robot name="sensor_d435" xmlns:xacro="http://ros.org/wiki/xacro">
-  <!-- Includes -->
-  <xacro:include filename="$(find realsense2_description)/urdf/_materials.urdf.xacro" />
-  <xacro:include filename="$(find realsense2_description)/urdf/_usb_plug.urdf.xacro" />
-  <xacro:macro name="sensor_d435"
-    params="parent *origin name:=camera use_nominal_extrinsics:=false add_plug:=false use_mesh:=true">
-    <xacro:property name="M_PI" value="3.1415926535897931" />
-    <!-- The following values are approximate, and the camera node
-     publishing TF values with actual calibrated camera extrinsic values -->
-    <xacro:property name="d435_cam_depth_to_infra1_offset" value="0.0" />
-    <xacro:property name="d435_cam_depth_to_infra2_offset" value="-0.050" />
-    <xacro:property name="d435_cam_depth_to_color_offset" value="0.015" />
-    <!-- The following values model the aluminum peripherial case for the
-  	D435 camera, with the camera joint represented by the actual
-  	peripherial camera tripod mount -->
-    <xacro:property name="d435_cam_width" value="0.090" />
-    <xacro:property name="d435_cam_height" value="0.025" />
-    <xacro:property name="d435_cam_depth" value="0.02505" />
-    <xacro:property name="d435_cam_mount_from_center_offset" value="0.0149" />
-    <!-- glass cover is 0.1 mm inwards from front aluminium plate -->
-    <xacro:property name="d435_glass_to_front" value="0.1e-3" />
-    <!-- see datasheet Revision 007, Fig. 4-4 page 65 -->
-    <xacro:property name="d435_zero_depth_to_glass" value="4.2e-3" />
-    <!-- convenience precomputation to avoid clutter-->
-    <xacro:property name="d435_mesh_x_offset"
-      value="${d435_cam_mount_from_center_offset-d435_glass_to_front-d435_zero_depth_to_glass}" />
-    <!-- The following offset is relative the the physical D435 camera peripherial
-  	camera tripod mount -->
-    <xacro:property name="d435_cam_depth_px" value="${d435_cam_mount_from_center_offset}" />
-    <xacro:property name="d435_cam_depth_py" value="0.0175" />
-    <xacro:property name="d435_cam_depth_pz" value="${d435_cam_height/2}" />
-    <!-- camera body, with origin at bottom screw mount -->
-    <joint name="${name}_joint" type="fixed">
-      <xacro:insert_block name="origin" />
-      <parent link="${parent}" />
-      <child link="${name}_bottom_screw_frame" />
-    </joint>
-    <link name="${name}_bottom_screw_frame" />
-    <joint name="${name}_link_joint" type="fixed">
-      <origin xyz="${d435_mesh_x_offset} ${d435_cam_depth_py} ${d435_cam_depth_pz}" rpy="0 0 0" />
-      <parent link="${name}_bottom_screw_frame" />
-      <child link="${name}_link" />
-    </joint>
-    <link name="${name}_link">
-      <visual>
-        <xacro:if value="${use_mesh}">
-          <!-- the mesh origin is at front plate in between the two infrared camera axes -->
-          <origin xyz="${d435_zero_depth_to_glass + d435_glass_to_front} ${-d435_cam_depth_py} 0"
-            rpy="${M_PI/2} 0 ${M_PI/2}" />
-          <geometry>
-            <mesh filename="file://$(find robot_description)/meshes/realsence_d435.dae" />
-          </geometry>
-        </xacro:if>
-        <xacro:unless value="${use_mesh}">
-          <origin xyz="0 ${-d435_cam_depth_py} 0" rpy="0 0 0" />
-          <geometry>
-            <box size="${d435_cam_depth} ${d435_cam_width} ${d435_cam_height}" />
-          </geometry>
-          <material name="aluminum" />
-        </xacro:unless>
-      </visual>
-      <collision>
-        <origin xyz="0 ${-d435_cam_depth_py} 0" rpy="0 0 0" />
-        <geometry>
-          <box size="${d435_cam_depth} ${d435_cam_width} ${d435_cam_height}" />
-        </geometry>
-      </collision>
-      <inertial>
-        <!-- The following are not reliable values, and should not be used for modeling -->
-        <mass value="0.0002" />
-        <origin xyz="0 0 0" />
-        <inertia ixx="0.0" ixy="0.0" ixz="0.0" iyy="0.0" iyz="0.0" izz="0.0" />
-      </inertial>
-    </link>
-    <!-- Use the nominal extrinsics between camera frames if the calibrated extrinsics aren't being
-    published. e.g. running the device in simulation  -->
-    <xacro:if value="${use_nominal_extrinsics}">
-      <!-- camera depth joints and links -->
-      <joint name="${name}_depth_joint" type="fixed">
-        <origin xyz="0 0 0" rpy="0 0 0" />
-        <parent link="${name}_link" />
-        <child link="${name}_depth_frame" />
-      </joint>
-      <link name="${name}_depth_frame" />
-      <joint name="${name}_depth_optical_joint" type="fixed">
-        <origin xyz="0 0 0" rpy="${-M_PI/2} 0 ${-M_PI/2}" />
-        <parent link="${name}_depth_frame" />
-        <child link="${name}_depth_optical_frame" />
-      </joint>
-      <link name="${name}_depth_optical_frame" />
-      <!-- camera left IR joints and links -->
-      <joint name="${name}_infra1_joint" type="fixed">
-        <origin xyz="0 ${d435_cam_depth_to_infra1_offset} 0" rpy="0 0 0" />
-        <parent link="${name}_link" />
-        <child link="${name}_infra1_frame" />
-      </joint>
-      <link name="${name}_infra1_frame" />
-      <joint name="${name}_infra1_optical_joint" type="fixed">
-        <origin xyz="0 0 0" rpy="${-M_PI/2} 0 ${-M_PI/2}" />
-        <parent link="${name}_infra1_frame" />
-        <child link="${name}_infra1_optical_frame" />
-      </joint>
-      <link name="${name}_infra1_optical_frame" />
-      <!-- camera right IR joints and links -->
-      <joint name="${name}_infra2_joint" type="fixed">
-        <origin xyz="0 ${d435_cam_depth_to_infra2_offset} 0" rpy="0 0 0" />
-        <parent link="${name}_link" />
-        <child link="${name}_infra2_frame" />
-      </joint>
-      <link name="${name}_infra2_frame" />
-      <joint name="${name}_infra2_optical_joint" type="fixed">
-        <origin xyz="0 0 0" rpy="${-M_PI/2} 0 ${-M_PI/2}" />
-        <parent link="${name}_infra2_frame" />
-        <child link="${name}_infra2_optical_frame" />
-      </joint>
-      <link name="${name}_infra2_optical_frame" />
-      <!-- camera color joints and links -->
-      <joint name="${name}_color_joint" type="fixed">
-        <origin xyz="0 ${d435_cam_depth_to_color_offset} 0" rpy="0 0 0" />
-        <parent link="${name}_link" />
-        <child link="${name}_color_frame" />
-      </joint>
-      <link name="${name}_color_frame" />
-      <joint name="${name}_color_optical_joint" type="fixed">
-        <origin xyz="0 0 0" rpy="${-M_PI/2} 0 ${-M_PI/2}" />
-        <parent link="${name}_color_frame" />
-        <child link="${name}_color_optical_frame" />
-      </joint>
-      <link name="${name}_color_optical_frame" />
+<robot xmlns:xacro="http://ros.org/wiki/xacro">
+    <xacro:if value="${add_realsense_d435}">
+        <xacro:arg name="use_nominal_extrinsics" default="true" />
+        <xacro:arg name="add_plug" default="false" />
+        <xacro:arg name="use_mesh" default="true" />
+        <xacro:include filename="$(find robot_description)/urdf/realsence_d435_macro.xacro" />
+        <xacro:arg name="add_rgbd" default="false" />
+        <xacro:property name="add_rgbd" value="$(arg add_rgbd)" />
+        <xacro:sensor_d435 parent="base_link" use_nominal_extrinsics="$(arg use_nominal_extrinsics)"
+            add_plug="$(arg add_plug)" use_mesh="$(arg use_mesh)">
+            <origin xyz="0.047 0 0.075" rpy="0 0 0" />
+        </xacro:sensor_d435>
     </xacro:if>
-    <xacro:if value="${add_plug}">
-      <xacro:usb_plug parent="${name}_link" name="${name}_usb_plug">
-        <origin
-          xyz="${d435_cam_mount_from_center_offset - 0.02095} ${-d435_cam_depth_py - 0.0353} 0"
-          rpy="0 0 0" />
-      </xacro:usb_plug>
-    </xacro:if>
-  </xacro:macro>
 </robot>

File: robot_description/urdf/rplidar_a2m8.xacro (robot description, xacro)
@@ -1,29 +1,31 @@
 <?xml version="1.0"?>
 <robot xmlns:xacro="http://ros.org/wiki/xacro">
-    <joint name="scan_joint" type="fixed">
-        <parent link="base_link" />
-        <child link="base_scan" />
-        <origin xyz="-0.032 0 0.124" rpy="0 0 0" />
-        <!-- <origin xyz="-0.032 0 0.184" rpy="0 0 0" /> -->
-    </joint>
-    <link name="base_scan">
-        <visual>
-            <origin xyz="0.005 0.03 -0.031" rpy="0 0 2.8" />
-            <geometry>
-                <mesh filename="file://$(find robot_description)/meshes/rplidar_a2m8.stl" scale="0.001 0.001 0.001" />
-            </geometry>
-            <material name="dark" />
-        </visual>
-        <collision>
-            <origin xyz="0.015 0 -0.0065" rpy="0 0 0" />
-            <geometry>
-                <cylinder length="0.0315" radius="0.055" />
-            </geometry>
-        </collision>
-        <inertial>
-            <mass value="0.114" />
-            <origin xyz="0 0 0" />
-            <inertia ixx="0.001" ixy="0.0" ixz="0.0" iyy="0.001" iyz="0.0" izz="0.001" />
-        </inertial>
-    </link>
+    <xacro:if value="${add_rplidar_a2}">
+        <joint name="scan_joint" type="fixed">
+            <parent link="base_link" />
+            <child link="base_scan" />
+            <origin xyz="-0.032 0 0.124" rpy="0 0 0" />
+        </joint>
+        <link name="base_scan">
+            <visual>
+                <origin xyz="0.005 0.03 -0.031" rpy="0 0 2.8" />
+                <geometry>
+                    <mesh filename="file://$(find robot_description)/meshes/rplidar_a2m8.stl"
+                        scale="0.001 0.001 0.001" />
+                </geometry>
+                <material name="dark" />
+            </visual>
+            <collision>
+                <origin xyz="0.015 0 -0.0065" rpy="0 0 0" />
+                <geometry>
+                    <cylinder length="0.0315" radius="0.055" />
+                </geometry>
+            </collision>
+            <inertial>
+                <mass value="0.114" />
+                <origin xyz="0 0 0" />
+                <inertia ixx="0.001" ixy="0.0" ixz="0.0" iyy="0.001" iyz="0.0" izz="0.001" />
+            </inertial>
+        </link>
+    </xacro:if>
 </robot>

File: robot_description/urdf/turtlebot3.urdf.xacro (robot description, xacro)
@@ -1,23 +1,12 @@
 <?xml version="1.0"?>
 <robot name="robot" xmlns:xacro="http://ros.org/wiki/xacro">
-	<material name="light_black">
-		<color rgba="0.4 0.4 0.4 1.0" />
-	</material>
-	<material name="dark">
-		<color rgba="0.3 0.3 0.3 1.0" />
-	</material>
+	<xacro:include filename="$(find robot_description)/urdf/robot_arguments.xacro" />
+	<xacro:include filename="$(find robot_description)/urdf/materials.xacro" />
 	<xacro:include filename="$(find robot_description)/urdf/robot_core.xacro" />
 	<xacro:include filename="$(find robot_description)/urdf/rplidar_a2m8.xacro" />
-	<xacro:include filename="$(find robot_description)/urdf/realsence_d435.gazebo.xacro" />
-	<xacro:include filename="$(find robot_description)/urdf/rplidar_a2m8.gazebo.xacro" />
-	<xacro:arg name="use_nominal_extrinsics" default="true" />
-	<xacro:arg name="add_plug" default="false" />
-	<xacro:arg name="use_mesh" default="true" />
 	<xacro:include filename="$(find robot_description)/urdf/realsence_d435.xacro" />
-	<xacro:sensor_d435 parent="base_link" use_nominal_extrinsics="$(arg use_nominal_extrinsics)"
-		add_plug="$(arg add_plug)" use_mesh="$(arg use_mesh)">
-		<origin xyz="0.047 0 0.075" rpy="0 0 0" />
-	</xacro:sensor_d435>
-	<xacro:arg name="namespace" default="" />
+	<!-- <xacro:include filename="$(find robot_description)/urdf/realsence_d435.gazebo.xacro" /> -->
+	<!-- <xacro:include filename="$(find robot_description)/urdf/rplidar_a2m8.gazebo.xacro" /> -->
+	<!-- <xacro:arg name="namespace" default="" />
 	<ros2_control name="GazeboSimSystem" type="system">
 		<hardware>
@@ -48,4 +37,4 @@
 			<parameters>$(find robot_simulation)/config/diff_drive_controller.yaml</parameters>
 		</plugin>
-	</gazebo>
+	</gazebo> -->
 </robot>

Commit message: Add simulation argument

File: robot_description/urdf/realsence_d435.xacro (robot description, xacro)
@@ -12,4 +12,27 @@
             <origin xyz="0.047 0 0.075" rpy="0 0 0" />
         </xacro:sensor_d435>
+        <xacro:if value="${simulation}">
+            <gazebo reference="camera_link">
+                <sensor name="rgbd_camera" type="rgbd_camera">
+                    <gz_frame_id>camera_link</gz_frame_id>
+                    <camera>
+                        <horizontal_fov>1.047</horizontal_fov>
+                        <image>
+                            <width>320</width>
+                            <height>240</height>
+                        </image>
+                        <clip>
+                            <near>0.1</near>
+                            <far>100</far>
+                        </clip>
+                    </camera>
+                    <always_on>1</always_on>
+                    <update_rate>50</update_rate>
+                    <visualize>true</visualize>
+                    <topic>rgbd_camera</topic>
+                    <enable_metrics>true</enable_metrics>
+                </sensor>
+            </gazebo>
+        </xacro:if>
     </xacro:if>
 </robot>

File: robot_description/urdf/robot_arguments.xacro (robot description, xacro)
@@ -1,7 +1,9 @@
 <?xml version="1.0"?>
 <robot xmlns:xacro="http://ros.org/wiki/xacro">
-    <xacro:arg name="add_rplidar_a2" default="false"/>
+    <xacro:arg name="add_rplidar_a2" default="true"/>
     <xacro:property name="add_rplidar_a2" value="$(arg add_rplidar_a2)" />
-    <xacro:arg name="add_realsense_d435" default="false"/>
+    <xacro:arg name="add_realsense_d435" default="true"/>
     <xacro:property name="add_realsense_d435" value="$(arg add_realsense_d435)" />
+    <xacro:arg name="simulation" default="false"/>
+    <xacro:property name="simulation" value="$(arg simulation)" />
 </robot>

File: robot_description/urdf/rplidar_a2m8.xacro (robot description, xacro)
@@ -28,4 +28,36 @@
             </inertial>
         </link>
+        <xacro:if value="${simulation}">
+            <gazebo reference="base_scan">
+                <sensor name='gpu_lidar' type='gpu_lidar'>
+                    <topic>scan</topic>
+                    <update_rate>10</update_rate>
+                    <gz_frame_id>base_scan</gz_frame_id>
+                    <lidar>
+                        <scan>
+                            <horizontal>
+                                <samples>640</samples>
+                                <resolution>1</resolution>
+                                <min_angle>-3.14</min_angle>
+                                <max_angle>3.14</max_angle>
+                            </horizontal>
+                            <vertical>
+                                <samples>16</samples>
+                                <resolution>1</resolution>
+                                <min_angle>-0.261799</min_angle>
+                                <max_angle>0.261799</max_angle>
+                            </vertical>
+                        </scan>
+                        <range>
+                            <min>0.08</min>
+                            <max>10.0</max>
+                            <resolution>0.01</resolution>
+                        </range>
+                    </lidar>
+                    <alwaysOn>1</alwaysOn>
+                    <visualize>true</visualize>
+                </sensor>
+            </gazebo>
+        </xacro:if>
     </xacro:if>
 </robot>

File: robot_description/urdf/turtlebot3.urdf.xacro (robot description, xacro)
@@ -6,6 +6,4 @@
 	<xacro:include filename="$(find robot_description)/urdf/rplidar_a2m8.xacro" />
 	<xacro:include filename="$(find robot_description)/urdf/realsence_d435.xacro" />
-	<!-- <xacro:include filename="$(find robot_description)/urdf/realsence_d435.gazebo.xacro" /> -->
-	<!-- <xacro:include filename="$(find robot_description)/urdf/rplidar_a2m8.gazebo.xacro" /> -->
 	<!-- <xacro:arg name="namespace" default="" />
 	<ros2_control name="GazeboSimSystem" type="system">
